File: hardware/DS2482-LC24XX-breakout.brd (EAGLE design)
At the start: 23.5 x 23.5 mm, 15 parts, among them IC1 DS2482-100S, IC2 EEPROM-I2CSMD, Q1 BSS84

Commit message: tweak gerbers
Parts:
- moved Q1 0.48 mm to (7.62, 8.41)
Connections:
- net N$2 renamed A0
- net N$3 renamed A1
- net N$4 renamed A2
- net N$5 renamed AD0
- net N$6 renamed AD1
Routing:
- net GND: track 21.9 -> 20.9 mm
- net N$1: track 10.9 -> 11.5 mm
Other:
- board text added: "A0"
- board text added: "A1"
- board text added: "A2"
- board text added: "AD0"
- board text added: "AD1"
