File: hardware/DS2482-LC24XX-breakout.sch (EAGLE design)
At the start: 14 parts, among them IC1 DS2482-100S, IC2 EEPROM-I2CSMD, Q1 BSS84

Commit message: tweak gerbers
Connections:
- net N$2 renamed A0
- net N$3 renamed A1
- net N$4 renamed A2
- net N$5 renamed AD0
- net N$6 renamed AD1
Changed lines of the file:
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@@
 </segment>
 </net>
-<net name="N$5" class="0">
+<net name="AD0" class="0">
 <segment>
 <pinref part="SJ1" gate="G$1" pin="2"/>
@@
 <pinref part="IC1" gate="G$1" pin="AD0"/>
 <wire x1="10.16" y1="55.88" x2="7.62" y2="55.88" width="0.1524" layer="91"/>
+<label x="10.16" y="55.88" size="1.778" layer="95"/>
 </segment>
 </net>
-<net name="N$6" class="0">
+<net name="AD1" class="0">
 <segment>
 <pinref part="SJ2" gate="G$1" pin="2"/>
@@
 <pinref part="IC1" gate="G$1" pin="AD1"/>
 <wire x1="20.32" y1="58.42" x2="7.62" y2="58.42" width="0.1524" layer="91"/>
+<label x="10.16" y="58.42" size="1.778" layer="95"/>
 </segment>
 </net>
-<net name="N$2" class="0">
+<net name="A0" class="0">
 <segment>
 <pinref part="SJ3" gate="G$1" pin="2"/>
@@
 <pinref part="IC2" gate="G$1" pin="A0"/>
 <wire x1="17.78" y1="96.52" x2="-17.78" y2="96.52" width="0.1524" layer="91"/>
+<label x="12.7" y="96.52" size="1.778" layer="95"/>
 </segment>
 </net>
-<net name="N$3" class="0">
+<net name="A1" class="0">
 <segment>
 <pinref part="IC2" gate="G$1" pin="A1"/>
@@
 <wire x1="17.78" y1="93.98" x2="-7.62" y2="93.98" width="0.1524" layer="91"/>
 <wire x1="-7.62" y1="93.98" x2="-7.62" y2="86.36" width="0.1524" layer="91"/>
+<label x="12.7" y="93.98" size="1.778" layer="95"/>
 </segment>
 </net>
-<net name="N$4" class="0">
+<net name="A2" class="0">
 <segment>
 <pinref part="IC2" gate="G$1" pin="A2"/>
@@
 <wire x1="17.78" y1="91.44" x2="2.54" y2="91.44" width="0.1524" layer="91"/>
 <wire x1="2.54" y1="91.44" x2="2.54" y2="88.9" width="0.1524" layer="91"/>
+<label x="12.7" y="91.44" size="1.778" layer="95"/>
 </segment>
 </net>
